File: Y11025HL-WIFI.kicad_pcb (KiCad board)
At the start: 2 copper layers, 50 x 47.5 mm, 66 parts, among them J1 Barrel_Jack_Switch_Pin3Ring, J2 Conn_01x05_Female, P1 JTAG, SW1 WIFI RST, U1 ESP-12E, U2 TLV767_DGN_ADJ, U3 TLV767_DRV_ADJ, U4 LM1117-3.3, U5 dspic33ep256gp502-QFN, U6 MIC5219-2.6

Commit message: .
Parts:
- moved G2 1.65 mm to (98.2, 117.8), turned to 0 degrees
- moved G5 0.48 mm to (105.5, 117.9)

Commit message: tp turned 90d
Parts:
- turned ML1 to 225 degrees
Routing:
- net SCL1: track 19.3 -> 23.9 mm
- net Net-(C14-Pad1): track 10.7 -> 14.7 mm, vias 0 -> 1
- net SDA1: track 19.7 -> 22.1 mm, vias 1 -> 2
- net GND: track 263.0 -> 264.3 mm, vias 11 -> 12
